Commit message: alleyhoop demo rviz

File: monitor/alleyhoop_monitor/urdf/alleyhoop.urdf (robot description, URDF)
Before this commit: robot alleyhoop, 2 links, 1 joints
Links:
- link base_link: geometry collision mesh filename=package://alleyhoop_monitor/meshes/AlleyHoopBaseLink.stl scale=0.0005 0.0005 0.0005; visual mesh filename=package://alleyhoop_monitor/meshes/AlleyHoopBaseLink.stl scale=0.0005 0.0005 0.0005
Joints:
- joint base_to_lidar: origin xyz=0 0 0.4 -> xyz=0 0 1

Commit message: lidar added in monitor demo

File: monitor/alleyhoop_monitor/urdf/alleyhoop.urdf (robot description, URDF)
Before this commit: robot alleyhoop, 2 links, 1 joints
Links:
- added link laser; visual cylinder length=0.1 radius=0.1
Joints:
- added joint lidar_to_laser: type fixed, parent base_link, child laser, origin xyz=0 0 1

Commit message: launch file fixed

File: monitor/alleyhoop_monitor/urdf/alleyhoop.urdf (robot description, URDF)
Before this commit: robot alleyhoop, 3 links, 2 joints
Links:
- removed link laser
Joints:
- removed joint lidar_to_laser

Commit message: urdf update && tf frames

File: monitor/alleyhoop_monitor/urdf/alleyhoop.urdf (robot description, URDF)
Before this commit: robot alleyhoop, 2 links, 1 joints
Links:
- added link laser
Joints:
- added joint lidar_link_to_laser: type fixed, parent lidar_link, child laser, origin xyz=0 0 0
- joint base_to_lidar: origin xyz=0 0 1 -> xyz=0 0 1.5
